File: obsidian_vault/03-design/03-3-tractor/03-3-4-ibt2/IBT-2_Gen2_Perf_Board.kicad_pcb (KiCad board)
At the start: 2 copper layers, 101.6 x 50.8 mm, 12 parts, among them J1_IBT2 wire/header pads, J2_DROK wire/header pads, J3_TEENSY wire/header pads

Commit message: Fix W6/W7 traces passing through R1/R2 5V pads
W6 (R_EN_NODE) and W7 (L_EN_NODE) were each drawn as a single segment
from col 2 to col 9, passing straight through R1/R2's 5V pad at col 5.
KiCad netlist saw this as a 5V <-> R_EN_NODE short.

Split each into two segments with a gap at col 4 -> col 6, leaving the
5V pad at col 5 isolated from the signal trace. Physically the insulated
wire still routes col 2 -> col 9 on the solder side; the gap just
prevents the false short in the KiCad netlist.

Co-Authored-By: Claude Sonnet 4.6 <noreply@anthropic.com>
Routing:
- net R_EN_NODE: track 88.9 -> 83.8 mm
- net L_EN_NODE: track 88.9 -> 83.8 mm
Changed lines of the file:
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@@
 	(segment
 		(start 101.98 95.48)
+		(end 107.06 95.48)
+		(width 0.6)
+		(layer "B.Cu")
+		(net 4)
+	)
+	(segment
+		(start 112.14 95.48)
 		(end 119.76 95.48)
 		(width 0.6)
@@
 	(segment
 		(start 101.98 87.86)
+		(end 107.06 87.86)
+		(width 0.6)
+		(layer "B.Cu")
+		(net 8)
+	)
+	(segment
+		(start 112.14 87.86)
 		(end 119.76 87.86)
 		(width 0.6)
